File: REF1027.kicad_sch (KiCad schematic)
At the start: 25 parts, among them Q1 ZVP2106A, Q2 BCX19, SW1 SW_SPDT, U2 27C256, U3 HY62256ALJ-10, U4 LZ95F45, U5 SN74HC32N, U6 SN74HC32N, U7 PALCE_20V8H-25JC/4

Commit message: Add files via upload
Other:
- note added: "PLD.Clk.OE = VCC PLD.Clk = (bits are BA7 to A0) - Write to 1xxxxxxx 1x1xxxx0 xx00xxxx D4 Pullup.OE = VCC /D4 Pullup = (bits are BA7 to A0) - Write to 1xxxxxxx 1x1xxxx0 xx00x11x (registered output) - Read from x0xxxxxx 0x213Fh A22.OE = VCC A22 = (bits are BA7 to A0) - Write to 1xxxxxxx 1x1xxxx0 xx00xxx1 (registered output) - Address is 1xxxxxxx xxxxxxxx xxxxxxxx SRAM.WE.OE=VCC /SRAM.WE= (bits are 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"
- note removed: "PLD.Clk.OE = VCC PLD.Clk = (bits are BA7 to A0) - Write to 1xxxxxxx 1x1xxxx0 xx00xxxx D4 Pullup.OE = VCC /D4 Pullup = (bits are BA7 to A0) - Write to 1xxxxxxx 1x1xxxx0 xx00xx1x (registered output) - Write to 1xxxxxxx 1x1xxxx0 xx00x1xx (registered output) - Read from x0xxxxxx 0x213Fh A22.OE = VCC A22 = (bits are BA7 to A0) - Write to 1xxxxxxx 1x1xxxx0 xx00xxx1 (registered output) - Address is 1xxx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"
- moved on the sheet: C4
Changed lines of the file:
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@@
 		)
 	)
-	(text "PLD.Clk.OE = VCC\nPLD.Clk = (bits are BA7 to A0)\n	- Write to 1xxxxxxx 1x1xxxx0 xx00xxxx\n\nD4 Pullup.OE = VCC\n/D4 Pullup = (bits are BA7 to A0)\n	- Write to 1xxxxxxx 1x1xxxx0 xx00xx1x (registered output)\n	- Write to 1xxxxxxx 1x1xxxx0 xx00x1xx (registered output)\n	- Read from x0xxxxxx 0x213Fh\n\nA22.OE = VCC\nA22 = (bits are BA7 to A0)\n	- Write to 1xxxxxxx 1x1xxxx0 xx00xxx1 (registered output)\n	- Address is 1xxxxxxx xxxxxxxx xxxxxxxx\n\nSRAM.WE.OE=VCC\n/SRAM.WE= (bits are BA7 to A0)\n	- Have not written to 1xxxxxxx 1x1xxxx0 xx00x1xx (registered output)\n	- For as long as Write is low\n\nD4 Pulldown.OE = VCC\nD4 Pulldown = (bits are BA7 to A0)\n	- Have not written to 1xxxxxxx 1x1xxxx0 xx00xx1x (registered output)\n	- Write to 1xxxxxxx 1x1xxxx0 xx00x1xx (registered output)\n	- Read from x1xxxxxx 0x213Fh"
+	(text "PLD.Clk.OE = VCC\nPLD.Clk = (bits are BA7 to A0)\n	- Write to 1xxxxxxx 1x1xxxx0 xx00xxxx\n\nD4 Pullup.OE = VCC\n/D4 Pullup = (bits are BA7 to A0)\n	- Write to 1xxxxxxx 1x1xxxx0 xx00x11x (registered output)\n	- Read from x0xxxxxx 0x213Fh\n\nA22.OE = VCC\nA22 = (bits are BA7 to A0)\n	- Write to 1xxxxxxx 1x1xxxx0 xx00xxx1 (registered output)\n	- Address is 1xxxxxxx xxxxxxxx xxxxxxxx\n\nSRAM.WE.OE=VCC\n/SRAM.WE= (bits are BA7 to A0)\n	- Have not written to 1xxxxxxx 1x1xxxx0 xx00x1xx (registered output)\n	- For as long as Write is low\n\nD4 Pulldown.OE = VCC\nD4 Pulldown = (bits are BA7 to A0)\n	- Write to 1xxxxxxx 1x1xxxx0 xx00x10x (registered output)\n	- Read from x1xxxxxx 0x213Fh"
 		(exclude_from_sim no)
 		(at 252.476 253.492 0)
@@
 	)
 	(label "GND"
-		(at 288.29 172.72 0)
+		(at 285.75 175.26 270)
 		(fields_autoplaced yes)
 		(effects
@@
 				(size 1.27 1.27)
 			)
-			(justify left bottom)
+			(justify right bottom)
 		)
 	)
@@
 	)
 	(label "VCC"
-		(at 283.21 172.72 180)
+		(at 285.75 170.18 90)
 		(fields_autoplaced yes)
 		(effects
@@
 				(size 1.27 1.27)
 			)
-			(justify right bottom)
+			(justify left bottom)
 		)
 	)
@@
 		(on_board yes)
 		(dnp no)
-		(fields_autoplaced yes)
 		(property "Reference" "D1"
-			(at 41.91 157.48 0)
+			(at 41.656 156.21 90)
 			(effects
 				(font
@@
 		)
 		(property "Value" "D_Filled"
-			(at 39.37 157.48 0)
+			(at 41.656 158.75 90)
 			(effects
 				(font
@@
 		(dnp no)
 		(property "Reference" "R1"
-			(at 60.96 116.84 90)
+			(at 62.23 115.57 0)
 			(effects
 				(font
@@
 		)
 		(property "Value" "332"
-			(at 63.5 116.84 90)
+			(at 62.23 118.11 0)
 			(effects
 				(font
@@
 		(on_board yes)
 		(dnp no)
-		(fields_autoplaced yes)
 		(property "Reference" "C2"
-			(at 57.15 143.5163 90)
+			(at 56.896 142.24 0)
 			(effects
 				(font
@@
 		)
 		(property "Value" "481 pF"
-			(at 54.61 143.5163 90)
+			(at 56.896 144.78 0)
 			(effects
 				(font
@@
 	(symbol
 		(lib_id "Device:C_Small")
-		(at 285.75 172.72 90)
+		(at 285.75 172.72 0)
 		(unit 1)
 		(exclude_from_sim no)
@@
 		(on_board yes)
 		(dnp no)
-		(fields_autoplaced yes)
 		(property "Reference" "C4"
-			(at 285.7563 166.37 90)
+			(at 292.862 171.704 0)
 			(effects
 				(font
@@
 		)
 		(property "Value" "100 nF"
-			(at 285.7563 168.91 90)
+			(at 292.862 174.244 0)
 			(effects
 				(font
@@
 		(on_board yes)
 		(dnp no)
-		(fields_autoplaced yes)
 		(property "Reference" "R2"
-			(at 60.96 143.51 90)
+			(at 71.12 142.24 0)
 			(effects
 				(font
@@
 		)
 		(property "Value" "473"
-			(at 63.5 143.51 90)
+			(at 71.12 144.78 0)
 			(effects
 				(font
@@
 		(dnp no)
 		(property "Reference" "R3"
-			(at 59.944 100.076 90)
+			(at 61.468 99.06 0)
 			(effects
 				(font
@@
 		)
 		(property "Value" "332"
-			(at 62.484 100.076 90)
+			(at 61.468 101.6 0)
 			(effects
 				(font
